File: TritLedSmdHysteresis/TritLedSmdHysteresis.kicad_pcb (KiCad board)
At the start: 2 copper layers, 22.2 x 16.5 mm, 15 parts, among them P1 Power, P2 In, U1 LM393

Commit message: Косметические процедуры
Signed-off-by: Алексей Кляузер <drum@pisem.net>
Parts:
- moved R7 1.27 mm to (41.9, 33.7)
Routing:
- net Net-(R7-Pad1): track 5.87 -> 7.14 mm
- net Net-(R5-Pad1): track 8.66 -> 9.93 mm
- net Net-(P2-Pad1): track 14.4 -> 13.1 mm
Other:
- board text added: "+"
- board text added: "+2,5"
- board text added: "-"
- board text added: "-2,5"
- board text added: "Trit"

Commit message: Расчёт сопротивлений
Signed-off-by: Алексей Кляузер <drum@pisem.net>
Parts:
- R1: value ?Ω -> 5,6Ω
- R2: value ?Ω -> 10КΩ
- R3: value ?Ω -> 22КΩ
- R4: value ?Ω -> 5,1КΩ
- R5, R6, R8: value ?Ω -> 4,7КΩ
- R7: value ?Ω -> 15КΩ
